File: Hardware/UniTest Board/UniTest Board.kicad_sch (KiCad schematic)
At the start: 0 parts

Commit message: add rpi to project
Other:
- added sheet MCU (untitled.kicad_sch)
Changed lines of the file:
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@@
 	(generator_version "9.0")
 	(paper "A4")
+	(sheet
+		(at 41.91 35.56)
+		(size 35.56 12.7)
+		(exclude_from_sim no)
+		(in_bom yes)
+		(on_board yes)
+		(dnp no)
+		(fields_autoplaced yes)
+		(stroke
+			(width 0.1524)
+			(type solid)
+		)
+		(fill
+			(color 0 0 0 0.0000)
+		)
+		(property "Sheetname" "MCU"
+			(at 41.91 34.8484 0)
+			(effects
+				(font
+					(size 1.27 1.27)
+				)
+				(justify left bottom)
+			)
+		)
+		(property "Sheetfile" "untitled.kicad_sch"
+			(at 41.91 48.8446 0)
+			(effects
+				(font
+					(size 1.27 1.27)
+				)
+				(justify left top)
+			)
+		)
+		(instances
+			(project "UniTest Board"
+				(path "/b4fc2485-daf0-4838-805a-f2c8e6577a31"
+					(page "2")
+				)
+			)
+		)
+	)
 	(sheet_instances
 		(path "/"
